File: kicad/Jabby.sch (KiCad schematic (older format))
At the start: 17 parts, among them J1 Conn_Ctrl_Pnl_01x04_Male, J2 Conn_GSM_01x05_Male, J3 Conn_Device_01x02_Male, Q1 2N2222, SW1 SW_DIP_x01, U1 MAX485E, U2 Mini360, U3 WeMos_D1_mini

Commit message: 0.2.9
Parts:
- added R7: 1K, symbol Device:R
Connections:
- net GND: now also R7.2
- net at J3.2 (Pin_2), U3.4 (SCK/D5): now also R7.1
Other:
- moved on the sheet: J3
Changed lines of the file:
@@
 	1    0    0    -1
 $EndComp
-Wire Wire Line
-	6200 5600 6200 5700
 NoConn ~ 5800 4400
 $Comp
@@
 L Connector:Conn_01x02_Male J3
 U 1 1 62104B7C
-P 8750 5500
-F 0 "J3" H 8900 5600 50  0000 R CNN
-F 1 "Conn_Device_01x02_Male" H 9250 5700 50  0000 R CNN
-F 2 "" H 8750 5500 50  0001 C CNN
-F 3 "~" H 8750 5500 50  0001 C CNN
-	1    8750 5500
+P 8850 5700
+F 0 "J3" H 9000 5800 50  0000 R CNN
+F 1 "Conn_Device_01x02_Male" H 9350 5900 50  0000 R CNN
+F 2 "" H 8850 5700 50  0001 C CNN
+F 3 "~" H 8850 5700 50  0001 C CNN
+	1    8850 5700
 	-1   0    0    1
 $EndComp
 Wire Wire Line
 	6600 4900 7150 4900
-Wire Wire Line
-	7150 4900 7150 5400
-Wire Wire Line
-	7150 5400 8550 5400
-Wire Wire Line
-	8550 5500 7150 5500
-Wire Wire Line
-	7150 5500 7150 5700
-Wire Wire Line
-	7150 5700 6200 5700
-Connection ~ 6200 5700
-Wire Wire Line
-	6200 5700 6200 5950
 NoConn ~ 6600 5200
 Text Label 8850 3850 0    50   ~ 0
@@
 Text Label 8850 4150 0    50   ~ 0
 TX
-Text Label 8850 5500 0    50   ~ 0
+Text Label 8950 5700 0    50   ~ 0
 COM
-Text Label 8850 5400 0    50   Italic 0
+Text Label 8950 5600 0    50   Italic 0
 XX
 NoConn ~ 6600 4800
@@
 Wire Wire Line
 	6900 4800 7300 4800
+$Comp
+L Device:R R7
+U 1 1 6271922F
+P 7150 5450
+F 0 "R7" H 7250 5500 50  0000 L CNN
+F 1 "1K" H 7250 5350 50  0000 L CNN
+F 2 "" V 7080 5450 50  0001 C CNN
+F 3 "~" H 7150 5450 50  0001 C CNN
+	1    7150 5450
+	1    0    0    -1
+$EndComp
+Wire Wire Line
+	8650 5700 7150 5700
+Wire Wire Line
+	7150 4900 7150 5300
+Wire Wire Line
+	7150 5300 8350 5300
+Wire Wire Line
+	8350 5300 8350 5600
+Wire Wire Line
+	8350 5600 8650 5600
+Wire Wire Line
+	6200 5600 6200 5700
+Connection ~ 7150 5300
+Wire Wire Line
+	7150 5600 7150 5700
+Wire Wire Line
+	7150 5700 6200 5700
+Connection ~ 7150 5700
+Connection ~ 6200 5700
+Wire Wire Line
+	6200 5700 6200 5950
 $EndSCHEMATC
